Commit message: Added support for gazebo simulation for the nano17 model only.

File: model/ft_sensor.urdf.xacro (robot description, xacro)
@@ -3,4 +3,5 @@
 	<!-- Include all available models -->
 	<xacro:include filename="$(find force_torque_sensor)/model/models.urdf.xacro"/>
+    <xacro:include filename="$(find force_torque_sensor)/model/ft_sensor.gazebo.xacro"/>
 	<!-- Base model for all sensor to have common frame names -->
 	<xacro:macro name="ft_sensor" params="parent name type *origin">
@@ -13,10 +14,15 @@
 			<insert_block name="nano17"/>
 		</link>
-		<joint name="${parent}_${name}_measure_joint" type="fixed">
+		<joint name="${parent}_${name}_measure_joint" type="revolute">
 			<insert_block name="nano17_measure_frame"/>
 			<parent link="${name}_${type}_base"/>
 			<child link="${name}_${type}_measure"/>
+			<limit lower="0" upper="0" effort="100" velocity="100"/>
+			<axis xyz="0 0 1" />
 		</joint>
-		<link name="${name}_${type}_measure"/>
+		<link name="${name}_${type}_measure">
+			<insert_block name="nano17_platform"/>
+		</link>
+        <xacro:ft_sensor_gazebo name="${name}" parent="${parent}" type="${type}"/>
 	</xacro:macro>
 </robot>

File: model/models.urdf.xacro (robot description, xacro)
@@ -40,4 +40,24 @@
 			</collision>
 	</xacro:property>
+	<xacro:property name="nano17_platform">
+			<inertial>
+				<mass value="0.002"/>
+				<origin xyz="0 0 0.0025"  />
+				<xacro:cylinder_inertia_def radius="0.085" length="0.005" mass="0.002"/>
+			</inertial>
+			<visual>
+				<!-- origin xyz="0 0 0.00725" rpy="0 0 0"/ -->
+				<origin xyz="0 0 0.0025" rpy="0 0 0"/>
+				<geometry>
+					<cylinder radius="0.0085" length="0.005"/>
+				</geometry>
+			</visual>
+			<collision>
+				<origin xyz="0 0 0.0025" rpy="0 0 0"/>
+				<geometry>
+					<cylinder radius="0.0085" length="0.005"/>
+				</geometry>
+			</collision>
+	</xacro:property>
 	<xacro:property name="nano17_measure_frame">
 		<origin xyz="0 0 0.0145" rpy="0 0 0"/>

Commit message: add F/T torque sensor and a cylinder test launch file now all seems work well !

File: model/ft_sensor.urdf.xacro (robot description, xacro)
@@ -12,8 +12,10 @@
 		</joint>
 		<link name="${name}_${type}_base">
-			<insert_block name="nano17"/>
+			<!-- <insert_block name="nano17"/> -->
+			<insert_block name="gamma"/>
 		</link>
 		<joint name="${parent}_${name}_measure_joint" type="revolute">
-			<insert_block name="nano17_measure_frame"/>
+			<!-- <insert_block name="nano17_measure_frame"/> -->
+			<insert_block name="gamma_measure_frame"/>
 			<parent link="${name}_${type}_base"/>
 			<child link="${name}_${type}_measure"/>
@@ -22,5 +24,6 @@
 		</joint>
 		<link name="${name}_${type}_measure">
-			<insert_block name="nano17_platform"/>
+			<!-- <insert_block name="nano17_platform"/> -->
+			<insert_block name="gamma_platform"/>
 		</link>
         <xacro:ft_sensor_gazebo name="${name}" parent="${parent}" type="${type}"/>

File: model/models.urdf.xacro (robot description, xacro)
@@ -63,3 +63,48 @@
 		<origin xyz="0 0 0.0145" rpy="0 0 0"/>
 	</xacro:property>
+<!-- http://www.ati-ia.com/products/ft/ft_models.aspx?id=Gamma -->
+<xacro:property name="gamma">
+			<inertial>
+				<mass value="0.255"/>
+				<origin xyz="0 0 0.01665"  />
+				<xacro:cylinder_inertia_def radius="0.0377" length="0.0333" mass="0.255"/>
+			</inertial>
+			<visual>
+				<!-- origin xyz="0 0 0.00725" rpy="0 0 0"/ -->
+				<origin xyz="0 0 0" rpy="0 0 0"/>
+				<geometry>
+					<!-- cylinder radius="0.0085" length="0.0145"/ -->
+					<mesh filename="package://force_torque_sensor/model/meshes/nano17.stl" scale="4.4 4.4 1"/>
+				</geometry>
+			</visual>
+			<collision>
+				<origin xyz="0 0 0.01665" rpy="0 0 0"/>
+				<geometry>
+					<cylinder radius="0.0377" length="0.005"/>
+				</geometry>
+			</collision>
+	</xacro:property>
+	<xacro:property name="gamma_platform">
+			<inertial>
+				<mass value="0.002"/>
+				<origin xyz="0 0 0.0025"  />
+				<xacro:cylinder_inertia_def radius="0.0377" length="0.005 " mass="0.255"/>
+			</inertial>
+			<visual>
+				<!-- origin xyz="0 0 0.00725" rpy="0 0 0"/ -->
+				<origin xyz="0 0 0.0025" rpy="0 0 0"/>
+				<geometry>
+					<cylinder radius="0.0377" length="0.005"/>
+				</geometry>
+			</visual>
+			<collision>
+				<origin xyz="0 0 0.0025" rpy="0 0 0"/>
+				<geometry>
+					<cylinder radius="0.0377" length="0.005"/>
+				</geometry>
+			</collision>
+	</xacro:property>
+	<xacro:property name="gamma_measure_frame">
+		<origin xyz="0 0 0.0145" rpy="0 0 0"/>
+	</xacro:property>
 </robot>

File: robot/nano17.urdf.xacro (robot description, xacro)
@@ -4,5 +4,9 @@
 	<xacro:include filename="$(find force_torque_sensor)/model/ft_sensor.urdf.xacro"/>
 	<link name="world"/>
+<!--
 	<xacro:ft_sensor parent="world" name="my_sensor" type="nano17">
+		<origin xyz="0 0 0" rpy="0 0 0"/>
+	</xacro:ft_sensor> -->
+	<xacro:ft_sensor parent="world" name="my_sensor" type="gamma">
 		<origin xyz="0 0 0" rpy="0 0 0"/>
 	</xacro:ft_sensor>
