Commit message: Try to add force torque sensor controller and visualization of force and torque

File: model/ft_sensor.gazebo.xacro (robot description, xacro)
@@ -20,5 +20,5 @@
           <type>gaussian</type>
           <mean>0.0</mean>
-          <stddev>0.003</stddev> <!-- change this to simulate noise -->
+          <stddev>0.003</stddev> <!-- change this to simulate noise  0.003-->
         </noise>
         </plugin>

File: model/ft_sensor.urdf.xacro (robot description, xacro)
@@ -20,5 +20,5 @@
 			<parent link="${name}_${type}_base"/>
 			<child link="${name}_${type}_measure"/>
-			<limit lower="0" upper="0" effort="100" velocity="100"/>
+			<limit lower="0" upper="0" effort="0" velocity="0"/>
 			<axis xyz="0 0 1" />
 		</joint>

Commit message: try to add force torque sensor controller [Status: failed]

File: model/ft_sensor.gazebo.xacro (robot description, xacro)
@@ -4,5 +4,6 @@
   <gazebo>
     <plugin name="gazebo_ros_control" filename="libgazebo_ros_control.so">
-      <robotNamespace>/${name}/</robotNamespace>
+       <robotNamespace>${name}</robotNamespace>
+       <robotSimType>gazebo_ros_control/DefaultRobotHWSim</robotSimType>
     </plugin>
   </gazebo>
@@ -18,5 +19,5 @@
     <!-- The ft_sensor plugin  -->
     <gazebo>
-        <plugin name="${name}_ft_sensor" filename="libgazebo_ros_ft_sensor.so">
+        <plugin name="ft_sensor" filename="libgazebo_ros_ft_sensor.so">
         <updateRate>1000.0</updateRate>
         <topicName>${parent}_${name}/ft_sensor_topic</topicName>

File: model/ft_sensor_gamma.urdf.xacro (robot description, xacro)
@@ -13,8 +13,8 @@
 		</joint>
 		<link name="${name}_${type}_base">
-		 <insert_block name="nano17"/>
+			<insert_block name="gamma"/>
 		</link>
 		<joint name="${parent}_${name}_measure_joint" type="revolute">
-			<insert_block name="nano17_measure_frame"/>
+			<insert_block name="gamma_measure_frame"/>
 			<parent link="${name}_${type}_base"/>
 			<child link="${name}_${type}_measure"/>
@@ -23,5 +23,5 @@
 		</joint>
 		<link name="${name}_${type}_measure">
-		 <insert_block name="nano17_platform"/>
+			<insert_block name="gamma_platform"/>
 		</link>
         <xacro:ft_sensor_gazebo name="${name}" parent="${parent}" type="${type}"/>

File: model/models.urdf.xacro (robot description, xacro)
@@ -75,5 +75,5 @@
 				<geometry>
 					<!-- cylinder radius="0.0085" length="0.0145"/ -->
-					<mesh filename="package://force_torque_sensor/model/meshes/nano17.stl" scale="4.4 4.4 1"/>
+					<mesh filename="package://force_torque_sensor/model/meshes/gamma.stl" scale="0.001 0.001 0.001"/>
 				</geometry>
 			</visual>
@@ -106,5 +106,5 @@
 	</xacro:property>
 	<xacro:property name="gamma_measure_frame">
-		<origin xyz="0 0 0.0145" rpy="0 0 0"/>
+		<origin xyz="0 0 0.0333" rpy="0 0 0"/>
 	</xacro:property>
 </robot>

File: robot/nano17.urdf.xacro (robot description, xacro)
@@ -4,9 +4,5 @@
 	<xacro:include filename="$(find force_torque_sensor)/model/ft_sensor.urdf.xacro"/>
 	<link name="world"/>
-<!--
 	<xacro:ft_sensor parent="world" name="my_sensor" type="nano17">
-		<origin xyz="0 0 0" rpy="0 0 0"/>
-	</xacro:ft_sensor> -->
-	<xacro:ft_sensor parent="world" name="my_sensor" type="gamma">
 		<origin xyz="0 0 0" rpy="0 0 0"/>
 	</xacro:ft_sensor>

Commit message: gamma support with hardware interface dedicate working: DONE only warning message to be solved

File: model/ft_sensor.gazebo.xacro (robot description, xacro)
@@ -2,10 +2,10 @@
 <robot xmlns:xacro="http://ros.org/wiki/xacro">
 	<xacro:macro name="ft_sensor_gazebo" params="parent name type">
-  <gazebo>
+<!--   <gazebo>
     <plugin name="gazebo_ros_control" filename="libgazebo_ros_control.so">
        <robotNamespace>${name}</robotNamespace>
        <robotSimType>gazebo_ros_control/DefaultRobotHWSim</robotSimType>
     </plugin>
-  </gazebo>
+  </gazebo>  -->
     <gazebo reference="${name}_${type}_base">
 			<gravity>true</gravity>

File: model/ft_sensor.trasmission.xacro (robot description, xacro)
@@ -4,17 +4,20 @@
 	<xacro:macro name="ft_sensor_transmission" params="parent name type">
       <ros>
-       <plugin name="force_torque_sensor_controller" filename="libforce_torque_sensor_controller.so">
+       <plugin name="force_torque_sensor" filename="libforce_torque_sensor_sim_ros_control.so">
         <!-- <plugin name="ros_controllers" filename="libforce_torque_sensor_controller.so">  -->
-          <robotNamespace>${name}</robotNamespace>
+          <robotNamespace>/${name}/</robotNamespace>
+              <joint name="${parent}_${name}_measure_joint">
+              <!-- <robotNamespace>/force_torque_sensor_sim_ros_control/</robotNamespace>   -->
+            <hardwareInterface>${Interface2}</hardwareInterface>
+       </joint>
        </plugin>
      </ros>
-   <ros>
+<!--    <ros>
    <transmission name="${parent}_${name}_trans">
         <robotNamespace>${name}</robotNamespace>
-        <type>transmission_interface/SimpleTransmission</type>
+        <type>${Interface2}</type>
       <joint name="${parent}_${name}_measure_joint">
         <robotNamespace>${name}</robotNamespace>
             <hardwareInterface>${Interface2}</hardwareInterface>
-            <hardwareInterface>EffortJointInterface</hardwareInterface>
        </joint>
       <actuator name="${name}_0_motor">
@@ -24,4 +27,5 @@
     </transmission>
   </ros>
+ -->
 	</xacro:macro>
 </robot>

File: model/ft_sensor_gamma.urdf.xacro (robot description, xacro)
@@ -19,5 +19,5 @@
 			<parent link="${name}_${type}_base"/>
 			<child link="${name}_${type}_measure"/>
-			<limit lower="0" upper="0" effort="0" velocity="0"/>
+ 			<limit lower="0" upper="0" effort="0" velocity="0"/>
 			<axis xyz="0 0 1" />
 		</joint>

Commit message: Merge nano17 e gamma sensor  add ft_simulation_display.launch

File: model/ft_sensor.gazebo.xacro (robot description, xacro)
@@ -8,11 +8,11 @@
     </plugin>
   </gazebo>  -->
-    <gazebo reference="${name}_${type}_base">
+    <gazebo reference="${name}_base">
 			<gravity>true</gravity>
 		</gazebo>
-		<gazebo reference="${name}_${type}_measure">
+		<gazebo reference="${name}_measure">
 			<gravity>true</gravity>
 		</gazebo>
-		<gazebo reference="${parent}_${name}_measure_joint">
+		<gazebo reference="${name}_measure_joint">
       <provideFeedback>true</provideFeedback>
     </gazebo>
@@ -21,6 +21,6 @@
         <plugin name="ft_sensor" filename="libgazebo_ros_ft_sensor.so">
         <updateRate>1000.0</updateRate>
-        <topicName>${parent}_${name}/ft_sensor_topic</topicName>
-        <jointName>${parent}_${name}_measure_joint</jointName>
+        <topicName>${name}/ft_sensor_topic</topicName>
+        <jointName>${name}_measure_joint</jointName>
         <noise>
           <type>gaussian</type>

File: model/ft_sensor.urdf.xacro (robot description, xacro)
@@ -7,20 +7,20 @@
 	<!-- Base model for all sensor to have common frame names -->
 	<xacro:macro name="ft_sensor" params="parent name type *origin">
-		<joint name="${parent}_${name}_base_joint" type="fixed">
+		<joint name="${name}_base_joint" type="fixed">
 			<insert_block name="origin"/>
 			<parent link="${parent}"/>
-			<child link="${name}_${type}_base"/>
+			<child link="${name}_base"/>
 		</joint>
-		<link name="${name}_${type}_base">
+		<link name="${name}_base">
 		 <insert_block name="nano17"/>
 		</link>
-		<joint name="${parent}_${name}_measure_joint" type="revolute">
+		<joint name="${name}_measure_joint" type="revolute">
 			<insert_block name="nano17_measure_frame"/>
-			<parent link="${name}_${type}_base"/>
-			<child link="${name}_${type}_measure"/>
+			<parent link="${name}_base"/>
+			<child link="${name}_measure"/>
 			<limit lower="0" upper="0" effort="0" velocity="0"/>
 			<axis xyz="0 0 1" />
 		</joint>
-		<link name="${name}_${type}_measure">
+		<link name="${name}_measure">
 		 <insert_block name="nano17_platform"/>
 		</link>

File: model/ft_sensor_gamma.urdf.xacro (robot description, xacro)
@@ -7,20 +7,20 @@
 	<!-- Base model for all sensor to have common frame names -->
 	<xacro:macro name="ft_sensor" params="parent name type *origin">
-		<joint name="${parent}_${name}_base_joint" type="fixed">
+		<joint name="${name}_base_joint" type="fixed">
 			<insert_block name="origin"/>
 			<parent link="${parent}"/>
-			<child link="${name}_${type}_base"/>
+			<child link="${name}_base"/>
 		</joint>
-		<link name="${name}_${type}_base">
+		<link name="${name}_base">
 			<insert_block name="gamma"/>
 		</link>
-		<joint name="${parent}_${name}_measure_joint" type="revolute">
+		<joint name="${name}_measure_joint" type="revolute">
 			<insert_block name="gamma_measure_frame"/>
-			<parent link="${name}_${type}_base"/>
-			<child link="${name}_${type}_measure"/>
+			<parent link="${name}_base"/>
+			<child link="${name}_measure"/>
  			<limit lower="0" upper="0" effort="0" velocity="0"/>
 			<axis xyz="0 0 1" />
 		</joint>
-		<link name="${name}_${type}_measure">
+		<link name="${name}_measure">
 			<insert_block name="gamma_platform"/>
 		</link>

File: robot/nano17.urdf.xacro (robot description, xacro)
@@ -1,4 +1,4 @@
 <?xml version="1.0"?>
-<robot xmlns:xacro="http://ros.org/wiki/xacro" name="nano17_example">
+<robot xmlns:xacro="http://ros.org/wiki/xacro" name="nano17">
 	<!-- Include the force-torque-sensor model -->
 	<xacro:include filename="$(find force_torque_sensor)/model/ft_sensor.urdf.xacro"/>

Commit message: improvement of hardware interface of force torque sensor

File: model/ft_sensor.gazebo.xacro (robot description, xacro)
@@ -9,8 +9,16 @@
   </gazebo>  -->
     <gazebo reference="${name}_base">
-			<gravity>true</gravity>
+<!-- 			<gravity>true</gravity>
+    <mu1>1</mu1>
+       <mu2>1</mu2>
+    <kp>100000</kp>
+    <kd>100.0</kd>  -->
 		</gazebo>
 		<gazebo reference="${name}_measure">
-			<gravity>true</gravity>
+<!--        <gravity>true</gravity>
+    <mu1>1</mu1>
+       <mu2>1</mu2>
+    <kp>100000</kp>
+    <kd>100.0</kd>  -->
 		</gazebo>
 		<gazebo reference="${name}_measure_joint">
@@ -30,4 +38,8 @@
         </plugin>
     </gazebo>
+    <ros>
+    <plugin name="filters" filename="libforce_torque_sensor_filter.so">
+   </plugin>
+   </ros>
 	</xacro:macro>
 </robot>

File: model/ft_sensor_gamma.urdf.xacro (robot description, xacro)
@@ -19,4 +19,5 @@
 			<parent link="${name}_base"/>
 			<child link="${name}_measure"/>
+			<dynamics damping="10.0" friction="10.0"/>
  			<limit lower="0" upper="0" effort="0" velocity="0"/>
 			<axis xyz="0 0 1" />

File: model/models.urdf.xacro (robot description, xacro)
@@ -88,10 +88,10 @@
 			<inertial>
 				<mass value="0.002"/>
-				<origin xyz="0 0 0.0025"  />
+				<origin xyz="0.0000 0 0.0025"  />
 				<xacro:cylinder_inertia_def radius="0.0377" length="0.005 " mass="0.255"/>
 			</inertial>
 			<visual>
 				<!-- origin xyz="0 0 0.00725" rpy="0 0 0"/ -->
-				<origin xyz="0 0 0.0025" rpy="0 0 0"/>
+				<origin xyz="0.0000 0 0.0025" rpy="0 0 0"/>
 				<geometry>
 					<cylinder radius="0.0377" length="0.005"/>
@@ -99,5 +99,5 @@
 			</visual>
 			<collision>
-				<origin xyz="0 0 0.0025" rpy="0 0 0"/>
+				<origin xyz="0.0000 0 0.0025" rpy="0 0 0"/>
 				<geometry>
 					<cylinder radius="0.0377" length="0.005"/>
@@ -106,5 +106,5 @@
 	</xacro:property>
 	<xacro:property name="gamma_measure_frame">
-		<origin xyz="0 0 0.0333" rpy="0 0 0"/>
+		<origin xyz="0.0000 0 0.0333" rpy="0 0 0"/>
 	</xacro:property>
 </robot>

File: robot/cylinder.urdf.xacro (robot description, xacro)
@@ -12,10 +12,10 @@
 			<!-- solid cylinder : Izz=(m*r^2)/2; Ixx=Iyy=1/12*m*(3*r^2+h^2) -->
 			<!-- <inertia  ixx="0.002385" ixy="0.00"  ixz="0.00" iyy="0.002385" iyz="0.00" izz="0.00027" /> -->
-				<mass value="0.3"/>
+				<mass value="0.6"/>
 				<origin xyz="0 0 0.15"  />
-				<xacro:cylinder_inertia_def radius="0.03" length="0.3" mass="0.3" />
+				<xacro:cylinder_inertia_def radius="0.03" length="0.3" mass="0.6" />
 		</inertial>
 		<visual>
-			<origin xyz="0 0 0" rpy="0 0 0"/>
+			<origin xyz="0 0 0.15" rpy="0 0 0"/>
 			<geometry>
 				<cylinder length="0.3" radius="0.03"/>
@@ -23,5 +23,5 @@
 		</visual>
 		<collision>
-			<origin xyz="0 0 0" rpy="0 0 0"/>
+			<origin xyz="0 0 0.15" rpy="0 0 0"/>
 			<geometry>
 				<cylinder length="0.3" radius="0.03"/>
@@ -30,10 +30,11 @@
 	</link>
 	<gazebo reference="cylinder">
-		<!-- <selfCollide>true</selfCollide -->
+		 <selfCollide>true</selfCollide>
+        	  <!-- <maxContacts>1</maxContacts>   -->
 	     <gravity>true</gravity>
-		<mu1>0.6</mu1>
-	     <mu2>0.6</mu2>
-		<kp>10000.0</kp>
-	  <kd>100.0</kd>
+ 		<mu1>1</mu1>
+	     <mu2>1</mu2>
+		<kp>100000</kp>
+	  <kd>1000.0</kd>
 	 </gazebo>
 </robot>

Commit message: final version force torque sensor

File: model/ft_sensor.gazebo.xacro (robot description, xacro)
@@ -9,20 +9,43 @@
   </gazebo>  -->
     <gazebo reference="${name}_base">
-<!-- 			<gravity>true</gravity>
-    <mu1>1</mu1>
+           <selfCollide>false</selfCollide>
+		</gazebo>
+       <gazebo reference="${name}_measure_joint">
+      <provideFeedback>true</provideFeedback>
+    </gazebo>
+    <gazebo reference="${name}_imu_joint">
+<!--       <provideFeedback>true</provideFeedback> -->
+    </gazebo>
+    <gazebo reference="${name}_imu_measure">
+      <material>Gazebo/Blue</material>
+     <sensor name='imu_sensor' type='imu'>
+        <always_on>1</always_on>
+        <update_rate>1000</update_rate>
+        <visualize>1</visualize>
+        <topic>__default_topic__</topic>
+        <imu/>
+        <plugin name='imu_plugin' filename='libgazebo_ros_imu_sensor.so'>
+    <topicName>${name}/imu</topicName>
+    <robotNamespace>${name}</robotNamespace>
+    <bodyName>${name}_imu_measure</bodyName>
+    <updateRateHZ>1000.0</updateRateHZ>
+    <!-- <gaussianNoise>0.0</gaussianNoise> -->
+    <gaussianNoise>0.003</gaussianNoise>
+    <xyzOffset>0.0 0.0 0.0</xyzOffset>
+    <rpyOffset>0.0 0.0 0.0</rpyOffset>
+        </plugin>
+      <pose>0 0 0 0 0 0</pose>
+      </sensor>
+    </gazebo>
+    <!-- <origin rpy="1.57 -1.57 -1.57" xyz="-0.0378 0 0.01665"/> -->
+    <gazebo reference="${name}_measure">
+            <selfCollide>false</selfCollide>
+            <!-- <maxContacts>1</maxContacts>   -->
+       <gravity>true</gravity>
+<!--    <mu1>1</mu1>
        <mu2>1</mu2>
     <kp>100000</kp>
-    <kd>100.0</kd>  -->
+    <kd>10.0</kd> -->
 		</gazebo>
-		<gazebo reference="${name}_measure">
-<!--        <gravity>true</gravity>
-    <mu1>1</mu1>
-       <mu2>1</mu2>
-    <kp>100000</kp>
-    <kd>100.0</kd>  -->
-		</gazebo>
-		<gazebo reference="${name}_measure_joint">
-      <provideFeedback>true</provideFeedback>
-    </gazebo>
     <!-- The ft_sensor plugin  -->
     <gazebo>
@@ -42,4 +65,8 @@
    </plugin>
    </ros>
+    <ros>
+     <plugin name="filters" filename="libimu_sensor_filter.so">
+     </plugin>
+   </ros>
 	</xacro:macro>
 </robot>

File: model/ft_sensor.trasmission.xacro (robot description, xacro)
@@ -6,4 +6,8 @@
           <robotNamespace>/${name}/</robotNamespace>
        </plugin>
+       	 <ros>
+           <plugin name="${name}_contact_point_estimato" filename="libcontact_point_estimator.so">
+	   </plugin>
+	 </ros>
 	</xacro:macro>
 </robot>

File: model/ft_sensor_gamma.urdf.xacro (robot description, xacro)
@@ -17,13 +17,26 @@
 		</link>
 		<joint name="${name}_measure_joint" type="revolute">
-			<insert_block name="gamma_measure_frame"/>
+		   <!--<origin rpy="0.0 0.0 0.0" xyz="0 0 0.0"/>-->
+		     <insert_block name="gamma_measure_frame"/>
 			<parent link="${name}_base"/>
 			<child link="${name}_measure"/>
-			<dynamics damping="10.0" friction="10.0"/>
+			<dynamics damping="0.0" friction="0.0"/>
  			<limit lower="0" upper="0" effort="0" velocity="0"/>
 			<axis xyz="0 0 1" />
 		</joint>
-		<link name="${name}_measure">
+         <link name="${name}_measure">
 			<insert_block name="gamma_platform"/>
+		</link>
+	 	<joint name="${name}_imu_joint" type="fixed">
+			<parent link="${name}_base"/>
+			<child link="${name}_imu_measure"/>
+			<axis xyz="0 0 1" />
+			<origin rpy="1.57 -1.57 -1.57" xyz="-0.0378 0 0.01665"/>
+<!-- 			<dynamics damping="10.0" friction="10.0"/>
+			 <limit lower="0" upper="0" effort="0" velocity="0"/>
+			<axis xyz="0 0 1" />  -->
+		</joint>
+         <link name="${name}_imu_measure">
+			<insert_block name="imu_platform"/>
 		</link>
         <xacro:ft_sensor_gazebo name="${name}" parent="${parent}" type="${type}"/>

File: model/models.urdf.xacro (robot description, xacro)
@@ -11,6 +11,12 @@
 	<xacro:macro name="cylinder_inertia_def" params="radius length mass">
 	<inertia ixx="${mass * (3 * radius * radius + length * length) / 12}"
-			 iyy="${mass * radius* radius / 2}"
-			 izz="${mass * (3 * radius * radius + length * length) / 12}"
+			 iyy="${mass * (3 * radius * radius + length * length) / 12}"
+			 izz="${mass * radius* radius / 2}"
+			 ixy="0" iyz="0" ixz="0"/>
+	</xacro:macro>
+    <xacro:macro name="box_inertia_def" params="h w d mass">
+	<inertia ixx="${mass * (w*w+d*d)/ 12}"
+			 iyy="${mass * (h*h+d*d)/ 12}"
+			 izz="${mass * (h*h+w*w) / 12}"
 			 ixy="0" iyz="0" ixz="0"/>
 	</xacro:macro>
@@ -42,7 +48,7 @@
 	<xacro:property name="nano17_platform">
 			<inertial>
-				<mass value="0.002"/>
+				<mass value="0.2"/>
 				<origin xyz="0 0 0.0025"  />
-				<xacro:cylinder_inertia_def radius="0.085" length="0.005" mass="0.002"/>
+				<xacro:cylinder_inertia_def radius="0.085" length="0.005" mass="0.2"/>
 			</inertial>
 			<visual>
@@ -64,5 +70,5 @@
 	</xacro:property>
 <!-- http://www.ati-ia.com/products/ft/ft_models.aspx?id=Gamma -->
-<xacro:property name="gamma">
+  <xacro:property name="gamma">
 			<inertial>
 				<mass value="0.255"/>
@@ -87,13 +93,15 @@
 	<xacro:property name="gamma_platform">
 			<inertial>
-				<mass value="0.002"/>
+				<mass value="0.2"/>
 				<origin xyz="0.0000 0 0.0025"  />
-				<xacro:cylinder_inertia_def radius="0.0377" length="0.005 " mass="0.255"/>
+ 				<xacro:cylinder_inertia_def radius="0.0377" length="0.005 " mass="0.2"/>
+<!-- 				<xacro:cylinder_inertia_def radius="0.00377" length="0.005 " mass="0.002"/> -->
 			</inertial>
 			<visual>
-				<!-- origin xyz="0 0 0.00725" rpy="0 0 0"/ -->
-				<origin xyz="0.0000 0 0.0025" rpy="0 0 0"/>
+			      <origin xyz="0 0 0.0025" rpy="0 0 0"/>
+<!-- 				<origin xyz="0.0000 0 0.0025" rpy="0 0 0"/> -->
 				<geometry>
-					<cylinder radius="0.0377" length="0.005"/>
+ 					<cylinder radius="0.0377" length="0.005"/>
+<!-- 				        <cylinder radius="0.00377" length="0.005"/>  -->
 				</geometry>
 			</visual>
@@ -101,5 +109,6 @@
 				<origin xyz="0.0000 0 0.0025" rpy="0 0 0"/>
 				<geometry>
-					<cylinder radius="0.0377" length="0.005"/>
+ 					<cylinder radius="0.0377" length="0.005"/>
+<!-- 					<cylinder radius="0.00377" length="0.005"/> -->
 				</geometry>
 			</collision>
@@ -108,3 +117,22 @@
 		<origin xyz="0.0000 0 0.0333" rpy="0 0 0"/>
 	</xacro:property>
+ 	  <xacro:property name="imu_platform">
+           <inertial>
+				<mass value="0.005"/>
+					<origin xyz="0.00 0.0 0.0333" rpy="0 0 0"/>
+				<xacro:cuboid_inertia_def length="0.02" width="0.02" height="0.002" mass="0.005" />
+		</inertial>
+		<visual>
+				<origin xyz="0.0000 0.0 0.00" rpy="0 0 0"/>
+			 <geometry>
+		      <box size="0.02  0.02  0.002"/>
+			</geometry>
+		</visual>
+		<collision>
+			<origin xyz="0.0000 0.0 0.00" rpy="0 0 0"/>
+			<geometry>
+				<box size="0.02  0.02  0.002"/>
+			</geometry>
+		</collision>
+      </xacro:property>
 </robot>

File: robot/cylinder.urdf.xacro (robot description, xacro)
@@ -3,6 +3,6 @@
 	<xacro:macro name="cylinder_inertia_def" params="radius length mass">
 	<inertia ixx="${mass * (3 * radius * radius + length * length) / 12}"
-			 iyy="${mass * radius* radius / 2}"
-			 izz="${mass * (3 * radius * radius + length * length) / 12}"
+			 iyy="${mass * (3 * radius * radius + length * length) / 12}"
+			 izz="${mass * radius* radius / 2}"
 			 ixy="0" iyz="0" ixz="0"/>
 	</xacro:macro>
@@ -31,9 +31,9 @@
 	<gazebo reference="cylinder">
 		 <selfCollide>true</selfCollide>
-        	  <!-- <maxContacts>1</maxContacts>   -->
+        	  <maxContacts>100</maxContacts>
 	     <gravity>true</gravity>
  		<mu1>1</mu1>
 	     <mu2>1</mu2>
-		<kp>100000</kp>
+		<kp>100000000</kp>
 	  <kd>1000.0</kd>
 	 </gazebo>
