Commit message: Added real geometry of the nano17.

File: model/models.urdf.xacro (robot description, xacro)
@@ -26,7 +26,9 @@
 			</inertial>
 			<visual>
-				<origin xyz="0 0 0.00725" rpy="0 0 0"/>
+				<!-- origin xyz="0 0 0.00725" rpy="0 0 0"/ -->
+				<origin xyz="0 0 0" rpy="0 0 0"/>
 				<geometry>
-					<cylinder radius="0.0085" length="0.0145"/>
+					<!-- cylinder radius="0.0085" length="0.0145"/ -->
+					<mesh filename="package://force_torque_sensor/model/meshes/nano17.stl"/>
 				</geometry>
 			</visual>

Commit message: collision to match mesh

File: model/models.urdf.xacro (robot description, xacro)
@@ -36,5 +36,6 @@
 				<origin xyz="0 0 0.00725" rpy="0 0 0"/>
 				<geometry>
-					<cylinder radius="0.0085" length="0.0145"/>
+<!--					<cylinder radius="0.0085" length="0.0145"/>-->
+					<mesh filename="package://force_torque_sensor/model/meshes/nano17.stl"/>
 				</geometry>
 			</collision>

Commit message: collision amendment

File: model/models.urdf.xacro (robot description, xacro)
@@ -36,6 +36,6 @@
 				<origin xyz="0 0 0.00725" rpy="0 0 0"/>
 				<geometry>
-<!--					<cylinder radius="0.0085" length="0.0145"/>-->
-					<mesh filename="package://force_torque_sensor/model/meshes/nano17.stl"/>
+					<cylinder radius="0.0085" length="0.0145"/>
+<!--					<mesh filename="package://force_torque_sensor/model/meshes/nano17.stl"/>-->
 				</geometry>
 			</collision>
