Commit message: General Review of package.

File: robot/ft_sensor.urdf.xacro (robot description, xacro)
@@ -1,3 +1,4 @@
 <?xml version="1.0"?>
+<!-- nana17 -->
 <robot xmlns:xacro="http://www.ros.org/wiki/xacro" name="ft_sensor">
 	<!-- Include all available models -->
@@ -13,16 +14,15 @@
 		</joint>
 		<link name="${name}_base">
-			<insert_block name="gamma"/>
+		 <insert_block name="nano17"/>
 		</link>
 		<joint name="${name}_measure_joint" type="revolute">
-			<insert_block name="gamma_measure_frame"/>
+			<insert_block name="nano17_measure_frame"/>
 			<parent link="${name}_base"/>
 			<child link="${name}_measure"/>
-			<dynamics damping="10.0" friction="10.0"/>
- 			<limit lower="0" upper="0" effort="0" velocity="0"/>
+			<limit lower="0" upper="0" effort="0" velocity="0"/>
 			<axis xyz="0 0 1" />
 		</joint>
 		<link name="${name}_measure">
-			<insert_block name="gamma_platform"/>
+		 <insert_block name="nano17_platform"/>
 		</link>
         <xacro:ft_sensor_gazebo name="${name}" parent="${parent}" type="${type}"/>

File: robot/ft_sensor_gamma.urdf.xacro (robot description, xacro)
@@ -1,3 +1,4 @@
 <?xml version="1.0"?>
+<!-- gamma -->
 <robot xmlns:xacro="http://www.ros.org/wiki/xacro" name="ft_sensor">
 	<!-- Include all available models -->
@@ -13,15 +14,16 @@
 		</joint>
 		<link name="${name}_base">
-		 <insert_block name="nano17"/>
+			<insert_block name="gamma"/>
 		</link>
 		<joint name="${name}_measure_joint" type="revolute">
-			<insert_block name="nano17_measure_frame"/>
+			<insert_block name="gamma_measure_frame"/>
 			<parent link="${name}_base"/>
 			<child link="${name}_measure"/>
-			<limit lower="0" upper="0" effort="0" velocity="0"/>
+			<dynamics damping="10.0" friction="10.0"/>
+ 			<limit lower="0" upper="0" effort="0" velocity="0"/>
 			<axis xyz="0 0 1" />
 		</joint>
 		<link name="${name}_measure">
-		 <insert_block name="nano17_platform"/>
+			<insert_block name="gamma_platform"/>
 		</link>
         <xacro:ft_sensor_gazebo name="${name}" parent="${parent}" type="${type}"/>

File: robot/gamma.urdf.xacro (robot description, xacro)
@@ -2,5 +2,5 @@
 <robot xmlns:xacro="http://ros.org/wiki/xacro" name="gamma">
 	<!-- Include the force-torque-sensor model -->
-	<xacro:include filename="$(find force_torque_sensor)/model/ft_sensor_gamma.urdf.xacro"/>
+	<xacro:include filename="$(find force_torque_sensor)/robot/ft_sensor_gamma.urdf.xacro"/>
 	<link name="world"/>
 	<xacro:ft_sensor parent="world" name="my_sensor" type="gamma">

File: robot/nano17.urdf.xacro (robot description, xacro)
@@ -2,5 +2,5 @@
 <robot xmlns:xacro="http://ros.org/wiki/xacro" name="nano17">
 	<!-- Include the force-torque-sensor model -->
-	<xacro:include filename="$(find force_torque_sensor)/model/ft_sensor.urdf.xacro"/>
+	<xacro:include filename="$(find force_torque_sensor)/robot/ft_sensor.urdf.xacro"/>
 	<link name="world"/>
 	<xacro:ft_sensor parent="world" name="my_sensor" type="nano17">
